File: EL-Load-Digital/EL-Load-Digital.kicad_pcb (KiCad board)
At the start: 4 copper layers, 100 x 68.2 mm, 84 parts, among them J1 Conn_01x06_Male, J2 Conn_02x12_Counter_Clockwise, J3 Conn_01x05_Male, J4 Conn_02x12_Counter_Clockwise, J6 Imon, J7 Umon, J8 Conn_02x05_Odd_Even, J9 -5PWR, SW1 Pico Reset, U1 DAC8555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

Commit message: Digital PCB update
Parts:
- removed kibuzzard-635D1AE8: G***, kibuzzard-635D1AE8
- removed kibuzzard-635D1B7E: G***, kibuzzard-635D1B7E
- removed kibuzzard-635D1C19: G***, kibuzzard-635D1C19
- added C30: 100n, Capacitor_SMD:C_0805_2012Metric_Pad1.18x1.45mm_HandSolder, F.Cu at (104.2, 29.8)
- added J5: Conn_01x04_Pin, Connector_PinHeader_2.54mm:PinHeader_1x04_P2.54mm_Vertical, F.Cu at (85.7, 38.8)
- added JP2: Jumper_3_Bridged12, Jumper:SolderJumper-3_P1.3mm_Bridged2Bar12_RoundedPad1.0x1.5mm, F.Cu at (114.8, 28.4)
- added U13: 24LC64, Package_SO:SOIC-8_3.9x4.9mm_P1.27mm, F.Cu at (109.2, 28.9)
- added kibuzzard-64AAE6E2: G***, kibuzzard-64AAE6E2, F.Cu at (108.5, 47.7)
- added kibuzzard-64AAEA42: G***, kibuzzard-64AAEA42, F.Cu at (90.3, 53.9)
- added kibuzzard-64B1211E: G***, kibuzzard-64B1211E, F.Cu at (121.2, 47.7)
- added kibuzzard-64B12145: G***, kibuzzard-64B12145, F.Cu at (82.8, 34.9)
- moved J6 10.5 mm to (116.6, 69.1)
- moved J7 10.5 mm to (106.1, 69.1)
- moved C11 0.93 mm to (98.2, 28.1)
- moved R11 0.47 mm to (100.9, 73.0)
- moved R13 0.47 mm to (100.9, 70.9)
- moved R15 0.42 mm to (100.9, 68.8)
- moved C14 0.22 mm to (89.9, 37.8)
- moved C15 0.13 mm to (97.4, 67.0)
- moved U3 0.12 mm to (94.4, 65.7)
Connections:
- J2 pad 14: GND -> clampOff3V3
- J2 pad 3: GND -> GCOM
- J4 pad 14: GND -> clampOff3V3
- J4 pad 3: GND -> GCOM
- R2 pad 1: GND -> GCOM
- R4 pad 1: GND -> GCOM
- U12 pad 12: unconnected-(U12-GP2-Pad12) -> GP2
- U12 pad 13: unconnected-(U12-GP3-Pad13) -> GP3
- U12 pad 14: unconnected-(U12-GP4-Pad14) -> clampOff3V3
Routing:
- net GCOM: track 0.00 -> 65.7 mm, vias 0 -> 1
- net clampOff3V3: track 0.00 -> 59.2 mm, vias 0 -> 1
- net SCL: track 157.9 -> 183.4 mm, vias 5 -> 6
- net SDA: track 159.1 -> 182.7 mm, vias 3 -> 4
- net +3.3VD: track 152.5 -> 175.2 mm
- net Umon: track 78.1 -> 61.5 mm
- net +5V: track 227.0 -> 218.4 mm
- net Imon: track 61.7 -> 69.8 mm
- net GP3: track 0.00 -> 5.76 mm
- net GP2: track 0.00 -> 5.68 mm
- net OVPtriggered: track 41.8 -> 47.4 mm
- net Net-(JP2-C): track 0.00 -> 4.76 mm
- net ~{Von}: track 46.9 -> 49.4 mm
- net Vref: track 73.9 -> 74.9 mm
- net resetProt: track 45.0 -> 45.9 mm
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