File: EL-Load-Digital/EL-Load-Digital.kicad_sch (KiCad schematic)
At the start: 77 parts, among them J1 Conn_01x06_Male, J2 Conn_02x12_Counter_Clockwise, J3 Conn_01x05_Male, J4 Conn_02x12_Counter_Clockwise, J6 Imon, J7 Umon, J8 Conn_02x05_Odd_Even, J9 -5PWR, SW1 Pico Reset, U1 DAC8555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

Commit message: Digital PCB update
Parts:
- added C30: 100n, Capacitor_SMD:C_0805_2012Metric_Pad1.18x1.45mm_HandSolder, symbol Device:C_Small
- added J5: Conn_01x04_Pin, Connector_PinHeader_2.54mm:PinHeader_1x04_P2.54mm_Vertical, symbol Connector:Conn_01x04_Pin
- added JP2: Jumper_3_Bridged12, Jumper:SolderJumper-3_P1.3mm_Bridged2Bar12_RoundedPad1.0x1.5mm, symbol Jumper:Jumper_3_Bridged12
- added U13: 24LC64, Package_SO:SOIC-8_3.9x4.9mm_P1.27mm, symbol Memory_EEPROM:24LC64
- H1: now left out of the parts list
Connections:
- net +3.3VD: now also C30.1, JP2.3 (B), U13.8 (VCC)
- net GND: now also C30.2, J5.1 (Pin_1), JP2.1 (A), U13.2 (A1), U13.3 (A2), U13.4 (GND), U13.7 (WP); no longer J2.14 (Pin_14), J2.3 (Pin_3), J4.14 (Pin_14), J4.3 (Pin_3), R2.1, R4.1
- net SCL: now also U13.6 (SCL)
- net SDA: now also U13.5 (SDA)
- net GP2: now reaches U12.12 (GP2)
- net GP2: now also J5.2 (Pin_2)
- net GP3: now reaches U12.13 (GP3)
- net GP3: now also J5.3 (Pin_3)
- net clampOff3V3: now reaches U12.14 (GP4)
- net clampOff3V3: now also J2.14 (Pin_14), J4.14 (Pin_14)
- new net: JP2.2 (C), U13.1 (A0)
- new net GCOM: J2.3 (Pin_3), J4.3 (Pin_3), R2.1, R4.1
- no-connect marks 7 -> 5
