File: EL-Load-Analog/MCU.kicad_sch (KiCad schematic)
At the start: 2 parts, among them J4 Conn_02x08_Odd_Even, J8 Conn_02x08_Odd_Even

Commit message: Added snubber on input, bananajacks, sense connector, some cleanup.
Other:
- title: (none) -> Electronic Load Analog Test Board
Changed lines of the file:
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@@
 (kicad_sch (version 20230121) (generator eeschema)
   (paper "A4")
+  (title_block
+    (title "Electronic Load Analog Test Board")
+    (date "2023-12-30")
+    (rev "${VERSION}")
+    (comment 1 "License: CERN-OHL-W-2.0")
+  )
   (junction (at 61.595 74.295) (diameter 0) (color 0 0 0 0)
   )

Commit message: Added SenseError detection (including ocmponents), added clearances, fixed few BOM items.
Parts:
- J4: Part Name (none) -> H_Male_1x40_vertical_THT
- J8: Part Name (none) -> H_Female_2x8_SMD
Changed lines of the file:
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@@
-    (effects (font (size 1.27 1.27)) (justify left bottom))
-  )
-  (text "not implemented" (at 109.22 123.825 0)
     (effects (font (size 1.27 1.27)) (justify left bottom))
   )
@@
     )
     (property "Datasheet" "~" (at 80.645 71.755 0)
+      (effects (font (size 1.27 1.27)) hide)
+    )
+    (property "Part Name" "H_Male_1x40_vertical_THT" (at 80.645 71.755 0)
       (effects (font (size 1.27 1.27)) hide)
     )
@@
       (effects (font (size 1.27 1.27)) hide)
     )
+    (property "Part Name" "H_Female_2x8_SMD " (at 78.105 115.57 0)
+      (effects (font (size 1.27 1.27)) hide)
+    )
