File: EL-Load-Analog/dac_adc.kicad_sch (KiCad schematic)
At the start: 43 parts, among them U11 DAC8555, U12 DAC8555, U14 MCP6004, U18 MCP6V51, U19 MCP6V51, U20 ADS131M02

Commit message: Added snubber on input, bananajacks, sense connector, some cleanup.
Other:
- title: (none) -> Electronic Load Analog Test Board
Changed lines of the file:
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@@
 (kicad_sch (version 20230121) (generator eeschema)
   (paper "A4")
+  (title_block
+    (title "Electronic Load Analog Test Board")
+    (date "2023-12-30")
+    (rev "${VERSION}")
+    (comment 1 "License: CERN-OHL-W-2.0")
+  )
   (junction (at 33.655 170.18) (diameter 0) (color 0 0 0 0)
   )

Commit message: Added SenseError detection (including ocmponents), added clearances, fixed few BOM items.
Parts:
- C19, C20, C42, C44: Part Name (none) -> C_1.0uF_0805_20%
- C21, C22, C23, C24, C25, C26, C36, C37, C38, C39: Part Name (none) -> C_100.0nF_0805_20%
- C27, C28: Part Name (none) -> C_10.0uF_25V_X7R_10%_0805
- C30: footprint Capacitor_SMD:C_0805_2012Metric_Pad1.18x1.45mm_HandSolder -> Capacitor_SMD:C_0805_2012Metric; Part Name (none) -> C_1.0uF_0805_20%
- C40, C41: Part Name (none) -> C_10.0nF_0805_20%
- C45: Part Name (none) -> C_220.0nF_0805_20%
- D4, D5: Part Name (none) -> D_BAV99_SOT-23
- R24: footprint Resistor_SMD:R_0805_2012Metric_Pad1.20x1.40mm_HandSolder -> Resistor_SMD:R_0805_2012Metric; Part Name (none) -> R_2.0kΩ_0805_1%
- R25: footprint Resistor_SMD:R_0805_2012Metric_Pad1.20x1.40mm_HandSolder -> Resistor_SMD:R_0805_2012Metric; Part Name (none) -> R_10.0kΩ_0805_1%
- R26, R27, R30, R31: Part Name (none) -> R_100k_0805_0.1%
- R28, R29: Part Name (none) -> R_10k_0805_0.1%
- R32, R33, R34, R35: Part Name (none) -> R_1.0kΩ_0805_1%
- R36, R37, R38: Part Name (none) -> R_47.0Ω_0805_1%
- U11, U12: Part Name (none) -> U_DAC8555IPW
- U14: Part Name (none) -> U_MCP6004T
- U18, U19: Part Name (none) -> U_MCP6V51T-E/OT
- U20: Part Name (none) -> U_ADS131M02
