File: EL-Load-Analog/shifts-refs.kicad_sch (KiCad schematic)
At the start: 37 parts, among them U10 TL072/OPA2376, U16 TPS7A2030, U17 TPS72325, U21 LT1964-5, U22 AMS1117, U23 TLV1117-50, U4 REF5025AD

Commit message: Added SenseError detection (including ocmponents), added clearances, fixed few BOM items.
Parts:
- C10, C12, C29, C34, C503: Part Name (none) -> C_1.0uF_0805_20%
- C11, C34: Part Name (none) -> C_22u_16V_X5R_10%_0805
- C29: Part Name (none) -> C_2.2uF_10V_X7R_10%_0805
- C29: Part Name (none) -> C_10.0uF_25V_X7R_10%_0805
- C29, C33: Part Name (none) -> C_10.0nF_0805_20%
- C501, C502, C504, C505: Part Name (none) -> C_100.0nF_0805_20%
- R39: Part Name (none) -> R_91.0Ω_0805_1%
- R40: Part Name (none) -> R_1.8kΩ_0805_1%
- R41, R504: Part Name (none) -> R_220.0Ω_0805_1%
- R502, R507, R509: Part Name (none) -> R_10.0kΩ_0805_1%
- R503, R505: Part Name (none) -> R_15.0kΩ_0805_1%
- U10: Part Name (none) -> U_TL072CDT
- U16: Part Name (none) -> U_TPS7A2030PDBVR
- U17: Part Name (none) -> U_TPS72325DB
- U21: Part Name (none) -> U_LT1964ES5
- U22: Part Name (none) -> U_AZ1117CH-ADJTRG1
- U23: Part Name (none) -> U_AZ1117CH-5.0TRG1
- U4: Part Name (none) -> U_REF5025
Changed lines of the file:
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@@
+      (effects (font (size 1.27 1.27)) hide)
+    )
+    (property "Part Name" "C_1.0uF_0805_20%" (at 64.77 53.34 0)
       (effects (font (size 1.27 1.27)) hide)
     )
@@
     )
     (property "Datasheet" "~" (at 87.63 74.93 0)
+      (effects (font (size 1.27 1.27)) hide)
+    )
+    (property "Part Name" "R_15.0kΩ_0805_1%" (at 87.63 74.93 0)
       (effects (font (size 1.27 1.27)) hide)
     )
@@
       (effects (font (size 1.27 1.27)) hide)
     )
+    (property "Part Name" "C_2.2uF_10V_X7R_10%_0805" (at 113.03 165.1 0)
+      (effects (font (size 1.27 1.27)) hide)
+    )
     (pin "1")
     (pin "2")
@@
       (effects (font (size 1.27 1.27)) hide)
     )
+    (property "Part Name" "C_10.0nF_0805_20%" (at 109.22 184.785 0)
+      (effects (font (size 1.27 1.27)) hide)
+    )
     (pin "1")
     (pin "2")
@@
     )
     (property "Datasheet" "https://www.analog.com/media/en/technical-documentation/data-sheets/1964fb.pdf" (at 230.505 79.375 0)
+      (effects (font (size 1.27 1.27)) hide)
+    )
+    (property "Part Name" "U_LT1964ES5" (at 230.505 79.375 0)
       (effects (font (size 1.27 1.27)) hide)
     )
@@
       (effects (font (size 1.27 1.27)) hide)
     )
+    (property "Part Name" "C_10.0uF_25V_X7R_10%_0805" (at 255.27 73.025 0)
+      (effects (font (size 1.27 1.27)) hide)
+    )
     (pin "1")
     (pin "2")
@@
       (effects (font (size 1.27 1.27)) hide)
     )
+    (property "Part Name" "C_22u_16V_X5R_10%_0805" (at 265.43 38.735 0)
+      (effects (font (size 1.27 1.27)) hide)
+    )
     (pin "1")
     (pin "2")
@@
       (effects (font (size 1.27 1.27)) hide)
     )
+    (property "Part Name" "R_10.0kΩ_0805_1%" (at 129.54 74.93 0)
+      (effects (font (size 1.27 1.27)) hide)
+    )
     (pin "1")
     (pin "2")
@@
     )
     (property "Datasheet" "http://www.ti.com/lit/ds/symlink/tl071.pdf" (at 128.27 88.9 0)
+      (effects (font (size 1.27 1.27)) hide)
+    )
+    (property "Part Name" "U_TL072CDT " (at 128.27 88.9 0)
       (effects (font (size 1.27 1.27)) hide)
     )
@@
       (effects (font (size 1.27 1.27)) hide)
     )
+    (property "Part Name" "C_10.0uF_25V_X7R_10%_0805" (at 240.665 38.735 0)
+      (effects (font (size 1.27 1.27)) hide)
+    )
     (pin "1")
     (pin "2")
@@
       (effects (font (size 1.27 1.27)) hide)
     )
+    (property "Part Name" "R_220.0Ω_0805_1%" (at 208.915 50.8 0)
+      (effects (font (size 1.27 1.27)) hide)
+    )
     (pin "1")
     (pin "2")
@@
     )
     (property "Datasheet" "~" (at 208.915 44.45 0)
+      (effects (font (size 1.27 1.27)) hide)
+    )
+    (property "Part Name" "R_1.8kΩ_0805_1%" (at 208.915 44.45 0)
       (effects (font (size 1.27 1.27)) hide)
     )
@@
       (effects (font (size 1.27 1.27)) hide)
     )
+    (property "Part Name" "C_10.0nF_0805_20%" (at 204.47 50.8 0)
+      (effects (font (size 1.27 1.27)) hide)
+    )
     (pin "1")
     (pin "2")
@@
       (effects (font (size 1.27 1.27)) hide)
     )
+    (property "Part Name" "C_1.0uF_0805_20%" (at 54.61 52.07 0)
+      (effects (font (size 1.27 1.27)) hide)
+    )
     (pin "1")
     (pin "2")
@@
       (effects (font (size 1.27 1.27)) hide)
     )
+    (property "Part Name" "C_22u_16V_X5R_10%_0805" (at 73.66 53.34 0)
+      (effects (font (size 1.27 1.27)) hide)
+    )
     (pin "1")
     (pin "2")
@@
       (effects (font (size 1.27 1.27)) hide)
     )
+    (property "Part Name" "C_1.0uF_0805_20%" (at 73.025 136.525 0)
+      (effects (font (size 1.27 1.27)) hide)
+    )
     (pin "1")
     (pin "2")
@@
       (effects (font (size 1.27 1.27)) hide)
     )
+    (property "Part Name" "R_220.0Ω_0805_1%" (at 91.44 50.8 0)
+      (effects (font (size 1.27 1.27)) hide)
+    )
     (pin "1")
     (pin "2")
@@
     )
     (property "Datasheet" "http://www.ti.com/lit/ds/symlink/tlv1117.pdf" (at 252.73 34.925 0)
+      (effects (font (size 1.27 1.27)) hide)
+    )
+    (property "Part Name" "U_AZ1117CH-5.0TRG1" (at 252.73 34.925 0)
       (effects (font (size 1.27 1.27)) hide)
     )
@@
     (property "Datasheet" "http://www.ti.com/lit/ds/symlink/ref5030.pdf" (at 40.64 45.72 0)
       (effects (font (size 1.27 1.27) italic) hide)
+    )
+    (property "Part Name" "U_REF5025" (at 41.91 45.72 0)
+      (effects (font (size 1.27 1.27)) hide)
     )
     (pin "1")
@@
       (effects (font (size 1.27 1.27)) hide)
     )
+    (property "Part Name" "U_TL072CDT " (at 125.73 45.72 0)
+      (effects (font (size 1.27 1.27)) hide)
+    )
     (pin "1")
     (pin "2")
@@
       (effects (font (size 1.27 1.27)) hide)
     )
+    (property "Part Name" "R_10.0kΩ_0805_1%" (at 106.68 74.93 0)
+      (effects (font (size 1.27 1.27)) hide)
+    )
     (pin "1")
     (pin "2")
@@
       (effects (font (size 1.27 1.27)) hide)
     )
+    (property "Part Name" "C_100.0nF_0805_20%" (at 46.99 75.565 0)
+      (effects (font (size 1.27 1.27)) hide)
+    )
     (pin "1")
     (pin "2")
@@
     )
     (property "Datasheet" "~" (at 208.915 38.1 0)
+      (effects (font (size 1.27 1.27)) hide)
+    )
+    (property "Part Name" "R_91.0Ω_0805_1%" (at 208.915 38.1 0)
       (effects (font (size 1.27 1.27)) hide)
     )
@@
       (effects (font (size 1.27 1.27)) hide)
     )
+    (property "Part Name" "C_10.0uF_25V_X7R_10%_0805" (at 188.595 39.37 0)
+      (effects (font (size 1.27 1.27)) hide)
+    )
     (pin "1")
     (pin "2")
@@
       (effects (font (size 1.27 1.27)) hide)
     )
+    (property "Part Name" "C_100.0nF_0805_20%" (at 100.33 50.8 0)
+      (effects (font (size 1.27 1.27)) hide)
+    )
     (pin "1")
     (pin "2")
@@
     )
     (property "Datasheet" "" (at 92.71 167.005 0)
+      (effects (font (size 1.27 1.27)) hide)
+    )
+    (property "Part Name" "U_TPS72325DB " (at 93.98 174.625 0)
       (effects (font (size 1.27 1.27)) hide)
     )
@@
       (effects (font (size 1.27 1.27)) hide)
     )
+    (property "Part Name" "R_15.0kΩ_0805_1%" (at 91.44 82.55 0)
+      (effects (font (size 1.27 1.27)) hide)
+    )
     (pin "1")
     (pin "2")
@@
       (effects (font (size 1.27 1.27)) hide)
     )
+    (property "Part Name" "C_1.0uF_0805_20%" (at 109.855 136.525 0)
+      (effects (font (size 1.27 1.27)) hide)
+    )
     (pin "1")
     (pin "2")
@@
     )
     (property "Datasheet" "http://www.ti.com/lit/ds/symlink/tl071.pdf" (at 38.1 80.645 0)
+      (effects (font (size 1.27 1.27)) hide)
+    )
+    (property "Part Name" "U_TL072CDT " (at 38.1 80.645 0)
       (effects (font (size 1.27 1.27)) hide)
     )
@@
       (effects (font (size 1.27 1.27)) hide)
     )
+    (property "Part Name" "C_10.0nF_0805_20%" (at 244.475 73.025 0)
+      (effects (font (size 1.27 1.27)) hide)
+    )
     (pin "1")
     (pin "2")
@@
     )
     (property "Datasheet" "http://www.advanced-monolithic.com/pdf/ds1117.pdf" (at 203.2 41.91 0)
+      (effects (font (size 1.27 1.27)) hide)
+    )
+    (property "Part Name" "U_AZ1117CH-ADJTRG1 " (at 200.66 35.56 0)
       (effects (font (size 1.27 1.27)) hide)
     )
@@
       (effects (font (size 1.27 1.27)) hide)
     )
+    (property "Part Name" "C_22u_16V_X5R_10%_0805" (at 217.805 39.37 0)
+      (effects (font (size 1.27 1.27)) hide)
+    )
     (pin "1")
     (pin "2")
@@
     )
     (property "Datasheet" "" (at 93.345 130.175 0)
+      (effects (font (size 1.27 1.27)) hide)
+    )
+    (property "Part Name" "U_TPS7A2030PDBVR" (at 94.615 137.795 0)
       (effects (font (size 1.27 1.27)) hide)
     )
@@
       (effects (font (size 1.27 1.27)) hide)
     )
+    (property "Part Name" "R_10.0kΩ_0805_1%" (at 86.36 43.18 0)
+      (effects (font (size 1.27 1.27)) hide)
+    )
     (pin "1")
     (pin "2")
@@
       (effects (font (size 1.27 1.27)) hide)
     )
+    (property "Part Name" "C_100.0nF_0805_20%" (at 113.665 81.915 0)
+      (effects (font (size 1.27 1.27)) hide)
+    )
     (pin "1")
     (pin "2")
@@
       (effects (font (size 1.27 1.27)) hide)
     )
+    (property "Part Name" "C_2.2uF_10V_X7R_10%_0805" (at 79.375 163.83 0)
+      (effects (font (size 1.27 1.27)) hide)
+    )
     (pin "1")
     (pin "2")
@@
     )
     (property "Datasheet" "~" (at 22.86 45.085 0)
+      (effects (font (size 1.27 1.27)) hide)
+    )
+    (property "Part Name" "C_1.0uF_0805_20%" (at 22.86 45.085 0)
       (effects (font (size 1.27 1.27)) hide)
     )
@@
       (effects (font (size 1.27 1.27)) hide)
     )
+    (property "Part Name" "C_1.0uF_0805_20%" (at 211.455 72.39 0)
+      (effects (font (size 1.27 1.27)) hide)
+    )
     (pin "1")
     (pin "2")
@@
       (effects (font (size 1.27 1.27)) hide)
     )
+    (property "Part Name" "C_100.0nF_0805_20%" (at 46.99 85.725 0)
+      (effects (font (size 1.27 1.27)) hide)
+    )
