File: EL-Load-Power-MCU/MCU.kicad_sch (KiCad schematic)
At the start: 17 parts, among them J12 Conn_01x05_Pin, J9 SWD+UART header, Q1 BSS138, Q2 BSS138, SW1 Pico Reset, U11 24LC64, U6 MCP23017_SO, U8 SC0915

Commit message: Fixed Panel 1r1 and Power-MCU 2r2 versions
Parts:
- C9, C?: Part_Name (none) -> C_100.0nF_50V_0805_10%
- J12, J9: Consumable (none) -> 1; Part_Name (none) -> H_Male_1x40_vertical_THT
- Q1, Q2: Part_Name (none) -> Q_BSS138W
- R15, R16, R19, R20: Part_Name (none) -> R_3.0kΩ_0805_1%
- R17: Part_Name (none) -> R_20.0kΩ_0805_1%
- R21: Part_Name (none) -> R_10.0kΩ_0805_1%
- SW1: Part_Name (none) -> SW_SPST_NO_SMD_6x6x5mm
- U11: value 24LC64 -> 24C64; Part_Name (none) -> U_24C64
- U6: Part_Name (none) -> U_MCP23017-E/SO
- U8: Availability In Stock -> (none); Check_prices https://www.snapeda.com/parts/SC0915/Raspberry+Pi/view-part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 -> (none); MANUFACTURER Pi Supply -> (none); MF Raspberry Pi -> (none); MP SC0915 -> (none); MPN (none) -> SC0915; PARTREV 1.9 -> (none); Package None -> (none); Part_Name (none) -> EM_Raspberry_Pi_Pico; Price None -> (none); Purchase-URL https://www.snapeda.com/api/url_track_click_mouser/?unipart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 -> (none); SNAPEDA_PN SC0915 -> (none); STANDARD Manufacturer Recommendations -> (none); SnapEDA_Link https://www.snapeda.com/parts/SC0915/Raspberry+Pi/view-part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 -> (none)
Changed lines of the file:
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@@
+      (effects (font (size 1.27 1.27)) hide)
+    )
+    (property "Part_Name" "R_3.0kΩ_0805_1%" (at 181.61 59.69 0)
+      (effects (font (size 1.27 1.27)) hide)
+    )
+    (property "Consumable" "" (at 181.61 59.69 0)
+      (effects (font (size 1.27 1.27)) hide)
+    )
+    (property "Optional" "" (at 181.61 59.69 0)
       (effects (font (size 1.27 1.27)) hide)
     )
@@
     (property "MPN" "" (at 133.985 29.845 0)
       (effects (font (size 1.27 1.27)))
+    )
+    (property "Part_Name" "H_Male_1x40_vertical_THT " (at 133.985 29.845 0)
+      (effects (font (size 1.27 1.27)) hide)
+    )
+    (property "Consumable" "1" (at 133.985 29.845 0)
+      (effects (font (size 1.27 1.27)) hide)
+    )
+    (property "Optional" "" (at 133.985 29.845 0)
+      (effects (font (size 1.27 1.27)) hide)
     )
     (pin "1")
@@
       (effects (font (size 1.27 1.27)) hide)
     )
+    (property "Part_Name" "R_3.0kΩ_0805_1%" (at 208.28 40.005 0)
+      (effects (font (size 1.27 1.27)) hide)
+    )
+    (property "Consumable" "" (at 208.28 40.005 0)
+      (effects (font (size 1.27 1.27)) hide)
+    )
+    (property "Optional" "" (at 208.28 40.005 0)
+      (effects (font (size 1.27 1.27)) hide)
+    )
     (pin "1")
     (pin "2")
@@
       (effects (font (size 1.27 1.27)) hide)
     )
+    (property "Part_Name" "R_3.0kΩ_0805_1%" (at 127.635 79.375 0)
+      (effects (font (size 1.27 1.27)) hide)
+    )
+    (property "Consumable" "" (at 127.635 79.375 0)
+      (effects (font (size 1.27 1.27)) hide)
+    )
+    (property "Optional" "" (at 127.635 79.375 0)
+      (effects (font (size 1.27 1.27)) hide)
+    )
     (pin "1")
     (pin "2")
@@
       (effects (font (size 1.27 1.27)) hide)
     )
+    (property "Part_Name" "R_10.0kΩ_0805_1%" (at 175.895 83.185 0)
+      (effects (font (size 1.27 1.27)) hide)
+    )
+    (property "Consumable" "" (at 175.895 83.185 0)
+      (effects (font (size 1.27 1.27)) hide)
+    )
+    (property "Optional" "" (at 175.895 83.185 0)
+      (effects (font (size 1.27 1.27)) hide)
+    )
     (pin "1")
     (pin "2")
@@
     (property "MPN" "" (at 274.955 36.83 0)
       (effects (font (size 1.27 1.27)))
+    )
+    (property "Part_Name" "H_Male_1x40_vertical_THT " (at 274.955 36.83 0)
+      (effects (font (size 1.27 1.27)) hide)
+    )
+    (property "Consumable" "1" (at 274.955 36.83 0)
+      (effects (font (size 1.27 1.27)) hide)
+    )
+    (property "Optional" "" (at 274.955 36.83 0)
+      (effects (font (size 1.27 1.27)) hide)
     )
     (pin "2")
@@
       (effects (font (size 1.27 1.27)) hide)
     )
+    (property "Part_Name" "" (at 108.585 168.275 0)
+      (effects (font (size 1.27 1.27)) hide)
+    )
+    (property "Consumable" "" (at 108.585 168.275 0)
+      (effects (font (size 1.27 1.27)) hide)
+    )
+    (property "Optional" "" (at 108.585 168.275 0)
+      (effects (font (size 1.27 1.27)) hide)
+    )
     (pin "1")
     (pin "2")
@@
       (effects (font (size 1.27 1.27)) hide)
     )
+    (property "Part_Name" "R_3.0kΩ_0805_1%" (at 136.525 79.375 0)
+      (effects (font (size 1.27 1.27)) hide)
+    )
+    (property "Consumable" "" (at 136.525 79.375 0)
+      (effects (font (size 1.27 1.27)) hide)
+    )
+    (property "Optional" "" (at 136.525 79.375 0)
+      (effects (font (size 1.27 1.27)) hide)
+    )
     (pin "1")
     (pin "2")
@@
       (effects (font (size 1.27 1.27)) (justify left) hide)
     )
+    (property "Part_Name" "Q_BSS138W" (at 175.26 62.23 0)
+      (effects (font (size 1.27 1.27)) hide)
+    )
+    (property "Consumable" "" (at 175.26 62.23 0)
+      (effects (font (size 1.27 1.27)) hide)
+    )
+    (property "Optional" "" (at 175.26 62.23 0)
+      (effects (font (size 1.27 1.27)) hide)
+    )
     (pin "1")
     (pin "2")
@@
     )
     (property "Datasheet" "~" (at 22.225 50.165 0)
+      (effects (font (size 1.27 1.27)) hide)
+    )
+    (property "Part_Name" "SW_SPST_NO_SMD_6x6x5mm" (at 22.225 55.245 0)
+      (effects (font (size 1.27 1.27)) hide)
+    )
+    (property "Consumable" "" (at 22.225 55.245 0)
+      (effects (font (size 1.27 1.27)) hide)
+    )
+    (property "Optional" "" (at 22.225 55.245 0)
       (effects (font (size 1.27 1.27)) hide)
     )
@@
       (effects (font (size 1.27 1.27)) (justify left))
     )
-    (property "Value" "24LC64" (at 130.8609 163.83 0)
+    (property "Value" "24C64" (at 130.8609 163.83 0)
       (effects (font (size 1.27 1.27)) (justify left))
     )
@@
     )
     (property "Datasheet" "http://ww1.microchip.com/downloads/en/DeviceDoc/21189f.pdf" (at 128.905 170.815 0)
+      (effects (font (size 1.27 1.27)) hide)
+    )
+    (property "Part_Name" "U_24C64" (at 128.905 170.815 0)
+      (effects (font (size 1.27 1.27)) hide)
+    )
+    (property "Consumable" "" (at 128.905 170.815 0)
+      (effects (font (size 1.27 1.27)) hide)
+    )
+    (property "Optional" "" (at 128.905 170.815 0)
       (effects (font (size 1.27 1.27)) hide)
     )
@@
       (effects (font (size 1.27 1.27)) hide)
     )
+    (property "Part_Name" "R_20.0kΩ_0805_1%" (at 175.895 90.17 0)
+      (effects (font (size 1.27 1.27)) hide)
+    )
+    (property "Consumable" "" (at 175.895 90.17 0)
+      (effects (font (size 1.27 1.27)) hide)
+    )
+    (property "Optional" "" (at 175.895 90.17 0)
+      (effects (font (size 1.27 1.27)) hide)
+    )
     (pin "1")
     (pin "2")
@@
     (property "Datasheet" "http://ww1.microchip.com/downloads/en/DeviceDoc/20001952C.pdf" (at 250.19 110.49 0)
       (effects (font (size 1.27 1.27)) (justify left) hide)
+    )
+    (property "Part_Name" "U_MCP23017-E/SO" (at 245.11 82.55 0)
+      (effects (font (size 1.27 1.27)) hide)
+    )
+    (property "Consumable" "" (at 245.11 82.55 0)
+      (effects (font (size 1.27 1.27)) hide)
+    )
+    (property "Optional" "" (at 245.11 82.55 0)
+      (effects (font (size 1.27 1.27)) hide)
     )
     (pin "1")
@@
       (effects (font (size 1.27 1.27)))
     )
+    (property "Part_Name" "C_100.0nF_50V_0805_10%" (at 238.125 51.435 0)
+      (effects (font (size 1.27 1.27)) hide)
+    )
+    (property "Consumable" "" (at 238.125 51.435 0)
+      (effects (font (size 1.27 1.27)) hide)
+    )
+    (property "Optional" "" (at 238.125 51.435 0)
+      (effects (font (size 1.27 1.27)) hide)
+    )
     (pin "1")
     (pin "2")
@@
       (effects (font (size 1.27 1.27)) hide)
     )
-    (property "MF" "Raspberry Pi" (at 73.66 80.645 0)
+    (property "Description" "Raspberry Pi Pico Embedded Dev Module | Raspberry Pi SC0915" (at 73.66 80.645 0)
       (effects (font (size 1.27 1.27)) (justify bottom) hide)
     )
-    (property "Description" "\nRaspberry Pi Pico Embedded Dev Module | Raspberry Pi SC0915\n" (at 73.66 80.645 0)
-      (effects (font (size 1.27 1.27)) (justify bottom) hide)
-    )
-    (property "Package" "None" (at 73.66 80.645 0)
-      (effects (font (size 1.27 1.27)) (justify bottom) hide)
-    )
-    (property "Price" "None" (at 73.66 80.645 0)
-      (effects (font (size 1.27 1.27)) (justify bottom) hide)
-    )
-    (property "Check_prices" "https://www.snapeda.com/parts/SC0915/Raspberry+Pi/view-part/?ref=eda" (at 73.66 80.645 0)
-      (effects (font (size 1.27 1.27)) (justify bottom) hide)
-    )
-    (property "STANDARD" "Manufacturer Recommendations" (at 73.66 80.645 0)
-      (effects (font (size 1.27 1.27)) (justify bottom) hide)
-    )
-    (property "PARTREV" "1.9" (at 73.66 80.645 0)
-      (effects (font (size 1.27 1.27)) (justify bottom) hide)
-    )
-    (property "SnapEDA_Link" "https://www.snapeda.com/parts/SC0915/Raspberry+Pi/view-part/?ref=snap" (at 73.66 80.645 0)
-      (effects (font (size 1.27 1.27)) (justify bottom) hide)
-    )
-    (property "MP" "SC0915" (at 73.66 80.645 0)
-      (effects (font (size 1.27 1.27)) (justify bottom) hide)
-    )
-    (property "Purchase-URL" "https://www.snapeda.com/api/url_track_click_mouser/?unipart_id=6331605&manufacturer=Raspberry Pi&part_name=SC0915&search_term=raspberry pi pico" (at 73.66 80.645 0)
-      (effects (font (size 1.27 1.27)) (justify bottom) hide)
-    )
-    (property "MANUFACTURER" "Pi Supply" (at 73.66 80.645 0)
-      (effects (font (size 1.27 1.27)) (justify bottom) hide)
-    )
-    (property "Availability" "In Stock" (at 73.66 80.645 0)
-      (effects (font (size 1.27 1.27)) (justify bottom) hide)
-    )
-    (property "SNAPEDA_PN" "SC0915" (at 73.66 80.645 0)
-      (effects (font (size 1.27 1.27)) (justify bottom) hide)
-    )
-    (property "MPN" "" (at 73.66 80.645 0)
-      (effects (font (size 1.27 1.27)))
+    (property "MPN" "SC0915" (at 73.66 80.645 0)
+      (effects (font (size 1.27 1.27)))
+    )
+    (property "Part_Name" "EM_Raspberry_Pi_Pico " (at 73.66 80.645 0)
+      (effects (font (size 1.27 1.27)) hide)
+    )
+    (property "Consumable" "" (at 73.66 80.645 0)
+      (effects (font (size 1.27 1.27)) hide)
+    )
+    (property "Optional" "" (at 73.66 80.645 0)
+      (effects (font (size 1.27 1.27)) hide)
     )
     (pin "1")
@@
       (effects (font (size 1.27 1.27)) (justify left) hide)
     )
+    (property "Part_Name" "Q_BSS138W" (at 201.93 42.545 0)
+      (effects (font (size 1.27 1.27)) hide)
+    )
+    (property "Consumable" "" (at 201.93 42.545 0)
+      (effects (font (size 1.27 1.27)) hide)
+    )
+    (property "Optional" "" (at 201.93 42.545 0)
+      (effects (font (size 1.27 1.27)) hide)
+    )
     (pin "1")
     (pin "2")
@@
       (effects (font (size 1.27 1.27)) hide)
     )
+    (property "Part_Name" "C_100.0nF_50V_0805_10%" (at 97.155 170.18 0)
+      (effects (font (size 1.27 1.27)) hide)
+    )
+    (property "Consumable" "" (at 97.155 170.18 0)
+      (effects (font (size 1.27 1.27)) hide)
+    )
+    (property "Optional" "" (at 97.155 170.18 0)
+      (effects (font (size 1.27 1.27)) hide)
+    )

Commit message: Fixes to Power-MCU board.
Other:
- title: EL-Load-PowerTest2 -> EL-Load-Power-MCU
Changed lines of the file:
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@@
   (paper "A4")
   (title_block
-    (title "EL-Load-PowerTest2")
-    (date "2023-11-28")
+    (title "EL-Load-Power-MCU")
+    (date "2024-02-04")
     (rev "${VERSION}r${PCBVERSION}")
   )

Commit message: Working on #4,#2 fixed #8,#22
Parts:
- Q1, Q2: value BSS138 -> BSS138W; footprint Package_TO_SOT_SMD:SOT-23 -> Package_TO_SOT_SMD:SOT-323_SC-70
Connections:
- net ~{VonLatch}: now also U6.28 (GPA7); no longer U6.21 (GPA0)
- net ~{Von}: now also U6.21 (GPA0); no longer U6.28 (GPA7)
Changed lines of the file:
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@@
     (effects (font (size 1.27 1.27)) (justify left))
   )
-  (hierarchical_label "~{Von}" (shape input) (at 265.43 102.87 0) (fields_autoplaced)
+  (hierarchical_label "~{Von}" (shape input) (at 265.43 85.09 0) (fields_autoplaced)
     (effects (font (size 1.27 1.27)) (justify left))
   )
@@
     (effects (font (size 1.27 1.27)) (justify right))
   )
-  (hierarchical_label "~{VonLatch}" (shape output) (at 265.43 85.09 0) (fields_autoplaced)
+  (hierarchical_label "~{VonLatch}" (shape output) (at 265.43 102.87 0) (fields_autoplaced)
     (effects (font (size 1.27 1.27)) (justify left))
   )
@@
       (effects (font (size 1.27 1.27)))
     )
-    (property "Value" "BSS138" (at 175.26 67.945 90)
-      (effects (font (size 1.27 1.27)))
-    )
-    (property "Footprint" "Package_TO_SOT_SMD:SOT-23" (at 173.355 67.31 0)
+    (property "Value" "BSS138W" (at 175.26 67.945 90)
+      (effects (font (size 1.27 1.27)))
+    )
+    (property "Footprint" "Package_TO_SOT_SMD:SOT-323_SC-70" (at 173.355 67.31 0)
       (effects (font (size 1.27 1.27) italic) (justify left) hide)
     )
-    (property "Datasheet" "https://www.onsemi.com/pub/Collateral/BSS138-D.PDF" (at 175.26 62.23 0)
+    (property "Datasheet" "https://www.diodes.com/assets/Datasheets/BSS138W.pdf" (at 175.26 62.23 0)
       (effects (font (size 1.27 1.27)) (justify left) hide)
     )
@@
     (property "Optional" "" (at 175.26 62.23 0)
       (effects (font (size 1.27 1.27)) hide)
+    )
+    (property "MPN" "" (at 175.26 62.23 0)
+      (effects (font (size 1.27 1.27)))
     )
     (pin "1")
@@
       (effects (font (size 1.27 1.27)))
     )
-    (property "Value" "BSS138" (at 201.93 48.26 90)
-      (effects (font (size 1.27 1.27)))
-    )
-    (property "Footprint" "Package_TO_SOT_SMD:SOT-23" (at 200.025 47.625 0)
+    (property "Value" "BSS138W" (at 201.93 48.26 90)
+      (effects (font (size 1.27 1.27)))
+    )
+    (property "Footprint" "Package_TO_SOT_SMD:SOT-323_SC-70" (at 200.025 47.625 0)
       (effects (font (size 1.27 1.27) italic) (justify left) hide)
     )
-    (property "Datasheet" "https://www.onsemi.com/pub/Collateral/BSS138-D.PDF" (at 201.93 42.545 0)
+    (property "Datasheet" "https://www.diodes.com/assets/Datasheets/BSS138W.pdf" (at 201.93 42.545 0)
       (effects (font (size 1.27 1.27)) (justify left) hide)
     )
@@
       (effects (font (size 1.27 1.27)) hide)
     )
-    (pin "1")
+    (property "MPN" "" (at 201.93 42.545 0)
+      (effects (font (size 1.27 1.27)))
+    )
+    (pin "1")

Commit message: EL-Load-Power-MCU PCB v4r4 release.
Parts:
- added BZ1: Buzzer, Buzzer_Beeper:Buzzer_12x9.5RM7.6, symbol Device:Buzzer
- added Q3: BSS138W, Package_TO_SOT_SMD:SOT-323_SC-70, symbol Transistor_FET:BSS138
- added R26, R27: 3k, Resistor_SMD:R_0805_2012Metric, symbol Device:R_Small
- added R31: 20k, Resistor_SMD:R_0805_2012Metric, symbol Device:R_Small
- added R5 (x2): 1k, Resistor_SMD:R_0805_2012Metric, symbol Device:R_Small
- C9, C?: Part_Name C_100.0nF_50V_0805_10% -> C_100.0nF_50V_0805_10%_X7R
- J12: footprint Connector_PinHeader_2.54mm:PinHeader_1x05_P2.54mm_Vertical -> Connector_PinHeader_2.54mm:PinHeader_1x03_P2.54mm_Vertical; symbol Connector:Conn_01x05_Pin -> Connector:Conn_01x03_Pin
Connections:
- net +3V3: now also J9.1 (Pin_1), R26.1, R27.1
- net +5VD: now also BZ1.1 (-), R5.1
- net DI-TP_CS: now also U8.24 (GP18); no longer U8.21 (GP16)
- net DI-TP_IRQ: now also U8.26 (GP20); no longer U8.22 (GP17)
- net EL-ADC_CS: now also U8.29 (GP22); no longer U8.26 (GP20)
- net GND: now also Q3.2 (S), R31.2
- net VoltSenseClear: now also U6.4 (GPB3); no longer U6.5 (GPB4)
- net ~{RESET}: now also U8.25 (GP19); no longer U8.24 (GP18)
- net ~{VonLatch}: now also U6.5 (GPB4); no longer U6.28 (GPA7)
- net HWGPIO_INT: now reaches R17.1, R21.2, U8.19 (GP14)
- net Buzzer: now reaches U6.3 (GPB2)
- net Buzzer: now also R5.1; no longer J12.4 (Pin_4)
- net EL-DAC_RDY renamed EL-ADC_RDY
- net SCL renamed HWIO_SCL
- net SDA renamed HWIO_SDA
- new net: BZ1.2 (+), Q3.3 (D), R5.2
- new net: Q3.1 (G), R31.1, R5.2
- new net KEYS_SCL: R27.2, U8.22 (GP17)
- new net KEYS_SDA: R26.2, U8.21 (GP16)
- new net reversePolarity: U6.28 (GPA7)
- no-connect marks 14 -> 11
Other:
- moved on the sheet: C9, JP7, Q2, R17, R20, R21, U11
