File: EL-Load-Power-MCU/standalone power.kicad_sch (KiCad schematic)
At the start: 11 parts, among them U10 MC34063AD

Commit message: EL-Load-Power-MCU PCB v4r4 release.
Parts:
- C25, C28: Part_Name (none) -> C_100uF_50V_Elec_8
- C27: value 200n -> 200p; Part_Name (none) -> C_200.0pF_0805_20%
- D17: value 1N5819WS -> SS14; Part_Name (none) -> D_SS14
- D18: Part_Name (none) -> D_Z_5V6_miniMELF
- F1: Part_Name (none) -> F_SMD_PTC_1A_1206
- L4: Part_Name (none) -> L_100uH_CD54
- R7: footprint Resistor_SMD:R_0805_2012Metric_Pad1.20x1.40mm_HandSolder -> Resistor_SMD:R_0805_2012Metric; Part_Name (none) -> R_0.33Ω_0805_1%
- U10: Part_Name (none) -> U_MC34063AD
Changed lines of the file:
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@@
       (effects (font (size 1.27 1.27)) (justify left))
     )
-    (property "Value" "1N5819WS" (at 157.48 82.8675 90)
+    (property "Value" "SS14" (at 157.48 82.8675 90)
       (effects (font (size 1.27 1.27)) (justify left))
     )
@@
       (effects (font (size 1.27 1.27)))
     )
+    (property "Part_Name" "D_SS14" (at 154.305 81.915 0)
+      (effects (font (size 1.27 1.27)) hide)
+    )
     (pin "1")
     (pin "2")
@@
       (effects (font (size 1.27 1.27)))
     )
-    (property "Footprint" "Resistor_SMD:R_0805_2012Metric_Pad1.20x1.40mm_HandSolder" (at 130.175 38.735 0)
+    (property "Footprint" "Resistor_SMD:R_0805_2012Metric" (at 130.175 38.735 0)
       (effects (font (size 1.27 1.27)) hide)
     )
@@
       (effects (font (size 1.27 1.27)) hide)
     )
-    (property "Part_Name" "" (at 130.175 38.735 0)
+    (property "Part_Name" "R_0.33Ω_0805_1%" (at 130.175 38.735 0)
       (effects (font (size 1.27 1.27)) hide)
     )
@@
       (effects (font (size 1.27 1.27)))
     )
+    (property "Part_Name" "C_100uF_50V_Elec_8" (at 176.53 80.01 0)
+      (effects (font (size 1.27 1.27)) hide)
+    )
     (pin "1")
     (pin "2")
@@
     )
     (property "Datasheet" "http://www.onsemi.com/pub_link/Collateral/MC34063A-D.PDF" (at 144.145 69.85 0)
+      (effects (font (size 1.27 1.27)) hide)
+    )
+    (property "Part_Name" "U_MC34063AD" (at 131.445 67.31 0)
       (effects (font (size 1.27 1.27)) hide)
     )
@@
       (effects (font (size 1.27 1.27)) hide)
     )
+    (property "Part_Name" "D_Z_5V6_miniMELF" (at 206.375 82.55 0)
+      (effects (font (size 1.27 1.27)) hide)
+    )
     (pin "2")
     (pin "1")
@@
       (effects (font (size 1.27 1.27)) (justify left))
     )
-    (property "Value" "200n" (at 113.03 81.9213 0)
+    (property "Value" "200p" (at 113.03 81.9213 0)
       (effects (font (size 1.27 1.27)) (justify left))
     )
@@
       (effects (font (size 1.27 1.27)))
     )
+    (property "Part_Name" "C_200.0pF_0805_20%" (at 110.49 80.645 0)
+      (effects (font (size 1.27 1.27)) hide)
+    )
     (pin "1")
     (pin "2")
@@
     )
     (property "Datasheet" "~" (at 165.735 72.39 0)
+      (effects (font (size 1.27 1.27)) hide)
+    )
+    (property "MPN" "" (at 165.735 72.39 0)
+      (effects (font (size 1.27 1.27)))
+    )
+    (property "Part_Name" "L_100uH_CD54" (at 165.735 72.39 0)
       (effects (font (size 1.27 1.27)) hide)
     )
@@
       (effects (font (size 1.27 1.27)))
     )
+    (property "Part_Name" "F_SMD_PTC_1A_1206" (at 83.82 38.735 0)
+      (effects (font (size 1.27 1.27)) hide)
+    )
     (pin "1")
     (pin "2")
@@
       (effects (font (size 1.27 1.27)))
     )
-    (pin "1")
+    (property "Part_Name" "C_100uF_50V_Elec_8" (at 99.06 62.23 0)
+      (effects (font (size 1.27 1.27)) hide)
+    )
+    (pin "1")
