File: EL-Load-Panel/EL-Load-Panel.kicad_sch (KiCad schematic)
At the start: 41 parts, among them J2 Conn_02x08_Odd_Even, J3 Touchscreen, SW1 ON/OFF, U1 MCP23008-xSO

Commit message: Added extra capacitor to Panel for stability. Upped schematic and pcb revisions to v2r3.
Parts:
- added C?: 10u, Capacitor_SMD:C_0805_2012Metric, symbol Device:C_Small
Connections:
- net +3V3: now also C?.1
- net GND: now also C?.2
Other:
- moved on the sheet: J3

Commit message: Initial Panel v3 commit
Parts:
- removed C?: 10u, Capacitor_SMD:C_0805_2012Metric, symbol Device:C_Small
- added C10, C9: 100n, Capacitor_SMD:C_0805_2012Metric, symbol Device:C_Small
- added C6, C8: 10u, Capacitor_SMD:CP_Elec_5x5.8, symbol Device:C_Polarized_Small
- added J3: Conn_01x04_Socket, Connector_Phoenix_MC:PhoenixContact_MCV_1,5_4-G-3.81_1x04_P3.81mm_Vertical, symbol Connector:Conn_01x04_Socket
- added U2: USBLC6-2SC6, Package_TO_SOT_SMD:SOT-23-6, symbol Power_Protection:USBLC6-2SC6
Connections:
- net +3V3: now also C10.1, C6.1, C8.1, C9.1, J3.4 (Pin_4), U2.5 (VBUS)
- net GND: now also C10.2, C6.2, C8.2, C9.2, J3.1 (Pin_1), U2.2 (GND)
- net SCL: now also U2.4 (I/O2)
- net SDA: now also U2.6 (I/O1)
- new net: J3.2 (Pin_2), U2.3 (I/O2)
- new net: J3.3 (Pin_3), U2.1 (I/O1)
Other:
- moved on the sheet: C3, C4, C5, C7, ENC1, J2, JP1, JP2, JP3, JP4, JP5, R1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
